File: HARDWARE/charger/MiniBot_charger_RevA.sch (KiCad schematic (older format))
At the start: 12 parts, among them CON1 CON8, U1 BL4054B-42TPRN(SOT23-5)

Commit message: Add files via upload
Other:
- note removed: "OPTION"
- moved on the sheet: BAT_CON1, C1, C2, CON1, LED1, R1, R2, R3, R4, R5, U1, USB1
